Commit message: update: IMu and Lidar works fine, but the camera not

File: src/final_project/urdf/imu.xacro (robot description, xacro)
@@ -3,7 +3,8 @@
     <gazebo reference="imu_link">
       <sensor type="imu" name="waffle_imu">
-        <always_on>true</always_on>
+        <always_on> 1 </always_on>
         <update_rate>200</update_rate>
         <topic> waffle_imu </topic>
+        <visualize> true </visualize>
         <imu>
           <angular_velocity>
@@ -48,5 +49,5 @@
           </linear_acceleration>
         </imu>
-        <plugin filename="ignition-gazebo-sensors-system" name="ignition::gazebo::systems::Sensors"/>
+        <plugin filename="ignition-gazebo-imu-system" name="ignition::gazebo::systems::Imu"/>
       </sensor>
     </gazebo>

File: src/final_project/urdf/waffle.urdf.xacro (robot description, xacro)
@@ -2,5 +2,9 @@
   <xacro:include filename="$(find final_project)/urdf/waffle.xacro" />
   <xacro:include filename="$(find final_project)/urdf/imu.xacro" />
+  <xacro:include filename="$(find final_project)/urdf/lidar.xacro" />
+  <xacro:include filename="$(find final_project)/urdf/camera.xacro" />
   <xacro:waffle/>
-  <!-- <xacro:waffle_imu/> -->
+  <xacro:waffle_imu/>
+  <xacro:waffle_lidar/>
+  <xacro:waffle_camera/>
 </robot>

File: src/final_project/urdf/waffle.xacro (robot description, xacro)
@@ -161,5 +161,6 @@
         <origin xyz="0.0 0 0.068" rpy="0 0 0"/>
     </joint>
-    <link name="imu_link"/>
+    <link name="imu_link">
+    </link>
     <joint name="scan_joint" type="fixed">
         <parent link="base_link"/>
@@ -168,6 +169,7 @@
     </joint>
     <link name="base_scan">
-        <visual>
-        <origin xyz="0 0 0" rpy="0 0 0"/>
+        <visual name="lidar_sensor_visual">
+        <origin xyz="0 0 0" rpy="0 0 0"/>
+        <!-- <pose>-0.064 0 0.121 0 0 0</pose> -->
         <geometry>
             <mesh filename="file://$(find final_project)/models/turtlebot3_common/meshes/lds.dae" scale="0.001 0.001 0.001"/>
@@ -175,16 +177,18 @@
         <material name="dark"/>
         </visual>
-        <collision>
-        <origin xyz="0.015 0 -0.0065" rpy="0 0 0"/>
-        <geometry>
-            <cylinder length="0.0315" radius="0.055"/>
-        </geometry>
-        </collision>
-        <inertial>
-        <mass value="0.114" />
-        <origin xyz="0 0 0" />
-        <inertia ixx="0.001" ixy="0.0" ixz="0.0"
-                iyy="0.001" iyz="0.0"
-                izz="0.001" />
+        <collision name="lidar_sensor_collision">
+            <!-- <pose>-0.052 0 0.111 0 0 0</pose> -->
+            <origin xyz="0.015 0 -0.0065" rpy="0 0 0"/>
+            <geometry>
+                <cylinder length="0.0315" radius="0.055"/>
+            </geometry>
+        </collision>
+        <inertial>
+            <pose>-0.052 0 0.111 0 0 0</pose>
+            <mass value="0.114" />
+            <origin xyz="0 0 0" />
+            <inertia ixx="0.001" ixy="0.0" ixz="0.0"
+                     iyy="0.001" iyz="0.0"
+                     izz="0.001" />
         </inertial>
     </link>
@@ -222,5 +226,6 @@
         <child link="camera_rgb_frame"/>
     </joint>
-    <link name="camera_rgb_frame"/>
+    <link name="camera_rgb_frame">
+    </link>
     <joint name="camera_rgb_optical_joint" type="fixed">
         <origin xyz="0 0 0" rpy="-1.57 0 -1.57"/>
@@ -243,4 +248,3 @@
     <link name="camera_depth_optical_frame"/>
   </xacro:macro>
-  <xacro:waffle/>
 </robot>
