Commit message: remap cmd_vel topic to /cmd_vel

File: src/final_project/urdf/turtlebot3_plugin.xacro (robot description, xacro)
@@ -1,4 +1,4 @@
 <robot xmlns:xacro="http://www.ros.org/wiki/xacro" name="waffle">
-  <xacro:macro name="turtlebot3_plugin">
+  <xacro:macro name="turtlebot3_plugin" params="entity_name">
     <gazebo>
       <plugin name="ignition::gazebo::systems::DiffDrive" filename="ignition-gazebo-diff-drive-system">
@@ -17,5 +17,5 @@
         <!-- <max_wheel_torque>20</max_wheel_torque> -->
         <max_angular_acceleration>1.0</max_angular_acceleration>
-        <topic>cmd_vel</topic>
+        <topic>${entity_name}/cmd_vel</topic>
         <!-- output -->
         <!-- <publish_odom>true</publish_odom> -->

File: src/final_project/urdf/waffle.urdf.xacro (robot description, xacro)
@@ -1,3 +1,4 @@
 <robot xmlns:xacro="http://www.ros.org/wiki/xacro"  name="waffle">
+  <xacro:arg name="entity_name" default="waffle"/>
   <xacro:include filename="$(find final_project)/urdf/waffle.xacro" />
   <xacro:include filename="$(find final_project)/urdf/imu.xacro" />
@@ -9,4 +10,4 @@
   <xacro:waffle_lidar/>
   <xacro:waffle_camera/>
-  <xacro:turtlebot3_plugin/>
+  <xacro:turtlebot3_plugin entity_name="$(arg entity_name)"/>
 </robot>
