Commit message: update the code such that it can spawn multiple waffle/burger bots!

File: src/final_project/urdf/burger.urdf.xacro (robot description, xacro)
@@ -1,4 +1,4 @@
-<robot xmlns:xacro="http://www.ros.org/wiki/xacro"  name="waffle">
-  <xacro:arg name="entity_name" default="waffle"/>
+<robot xmlns:xacro="http://www.ros.org/wiki/xacro"  name="burger">
+  <xacro:arg name="entity_name" default="burger"/>
   <xacro:include filename="$(find final_project)/urdf/waffle.xacro" />
   <xacro:include filename="$(find final_project)/urdf/imu.xacro" />
@@ -6,5 +6,4 @@
   <xacro:include filename="$(find final_project)/urdf/camera.xacro" />
   <xacro:include filename="$(find final_project)/urdf/turtlebot3_plugin.xacro" />
-  <xacro:include filename="$(find final_project)/urdf/ignition_system_plugin.xacro" />
   <xacro:waffle prefix="$(arg entity_name)"/>
   <xacro:waffle_imu prefix="$(arg entity_name)"/>
@@ -12,4 +11,3 @@
   <xacro:waffle_camera prefix="$(arg entity_name)"/>
   <xacro:turtlebot3_plugin entity_name="$(arg entity_name)"/>
-  <xacro:ignition_system_plugin/>
 </robot>

File: src/final_project/urdf/camera.xacro (robot description, xacro)
@@ -1,4 +1,4 @@
-<robot xmlns:xacro="http://www.ros.org/wiki/xacro" name="waffle">
-  <xacro:macro name="waffle_camera">
+<robot xmlns:xacro="http://www.ros.org/wiki/xacro">
+  <xacro:macro name="waffle_camera" params="prefix">
     <gazebo reference="camera_rgb_frame">
       <inertial>
@@ -15,9 +15,9 @@
       </inertial>
       <pose>0.069 -0.047 0.107 0 0 0</pose>
-      <sensor type="camera" name="waffle_camera">
+      <sensor type="camera" name="${prefix}_camera">
         <always_on> 1 </always_on>
         <visualize>true</visualize>
         <update_rate>30</update_rate>
-        <topic> waffle_camera </topic>
+        <topic> ${prefix}_camera </topic>
         <camera name="intel_realsense_r200">
           <horizontal_fov>1.02974</horizontal_fov>

File: src/final_project/urdf/imu.xacro (robot description, xacro)
@@ -1,9 +1,9 @@
-<robot xmlns:xacro="http://www.ros.org/wiki/xacro" name="waffle">
-  <xacro:macro name="waffle_imu">
+<robot xmlns:xacro="http://www.ros.org/wiki/xacro">
+  <xacro:macro name="waffle_imu" params="prefix">
     <gazebo reference="imu_link">
-      <sensor type="imu" name="waffle_imu">
+      <sensor type="imu" name="${prefix}_imu">
         <always_on> 1 </always_on>
         <update_rate>200</update_rate>
-        <topic> waffle_imu </topic>
+        <topic> ${prefix}_imu </topic>
         <visualize> true </visualize>
         <imu>

File: src/final_project/urdf/lidar.xacro (robot description, xacro)
@@ -1,11 +1,11 @@
-<robot xmlns:xacro="http://www.ros.org/wiki/xacro" name="waffle">
-  <xacro:macro name="waffle_lidar">
+<robot xmlns:xacro="http://www.ros.org/wiki/xacro">
+  <xacro:macro name="waffle_lidar" params="prefix">
     <gazebo reference="base_scan">
-      <sensor type="gpu_lidar" name="waffle_lidar">
+      <sensor type="gpu_lidar" name="${prefix}_lidar">
         <always_on> 1 </always_on>
         <visualize>true</visualize>
         <pose>-0.064 0 0.121 0 0 0</pose>
         <update_rate>5</update_rate>
-        <topic> waffle_lidar </topic>
+        <topic> ${prefix}_lidar </topic>
         <ignition_frame_id> base_scan </ignition_frame_id>
         <lidar>
@@ -31,7 +31,4 @@
       </sensor>
     </gazebo>
-    <gazebo>
-      <plugin filename="ignition-gazebo-sensors-system" name="ignition::gazebo::systems::Sensors"/>
-    </gazebo>
   </xacro:macro>
 </robot>

File: src/final_project/urdf/turtlebot3_plugin.xacro (robot description, xacro)
@@ -1,3 +1,3 @@
-<robot xmlns:xacro="http://www.ros.org/wiki/xacro" name="waffle">
+<robot xmlns:xacro="http://www.ros.org/wiki/xacro">
   <xacro:macro name="turtlebot3_plugin" params="entity_name">
     <gazebo>

File: src/final_project/urdf/waffle.urdf (robot description, URDF)
Before this commit: robot waffle, 13 links, 12 joints
Links:
- removed link base_footprint
- removed link base_link
- removed link base_scan
- removed link camera_depth_frame
- removed link camera_depth_optical_frame
- removed link camera_link
- removed link camera_rgb_frame
- removed link camera_rgb_optical_frame
- removed link caster_back_left_link
- removed link caster_back_right_link
- removed link imu_link
- removed link wheel_left_link
- removed link wheel_right_link
Joints:
- removed joint base_joint
- removed joint camera_depth_joint
- removed joint camera_depth_optical_joint
- removed joint camera_joint
- removed joint camera_rgb_joint
- removed joint camera_rgb_optical_joint
- removed joint caster_back_left_joint
- removed joint caster_back_right_joint
- removed joint imu_joint
- removed joint scan_joint
- removed joint wheel_left_joint
- removed joint wheel_right_joint

File: src/final_project/urdf/waffle.xacro (robot description, xacro)
@@ -1,4 +1,5 @@
-<robot xmlns:xacro="http://www.ros.org/wiki/xacro" name="waffle">
-  <xacro:macro name="waffle">
+<robot xmlns:xacro="http://www.ros.org/wiki/xacro">
+  <xacro:macro name="waffle" params="prefix">
+  <!-- <xacro:arg name="entity_name" default="waffle"/> -->
     <!-- Init colour -->
     <material name="black">
