Commit message: fixed issue: 1. xterm won't launch; 2. change scan_joint origin's z component from 0.122 to 0 (waffle.xacro line 200)

File: src/final_project/urdf/waffle.xacro (robot description, xacro)
@@ -167,5 +167,6 @@
         <parent link="base_link"/>
         <child link="base_scan"/>
-        <origin xyz="-0.064 0 0.122" rpy="0 0 0"/>
+        <!-- <origin xyz="-0.064 0 0.122" rpy="0 0 0"/> -->
+        <origin xyz="-0.064 0 0" rpy="0 0 0"/>
     </joint>
     <link name="base_scan">
