Commit message: fix bug: lidar in wrong position

File: src/final_project/urdf/lidar.xacro (robot description, xacro)
@@ -5,5 +5,6 @@
         <always_on> 1 </always_on>
         <visualize>true</visualize>
-        <pose>-0.064 0 0.121 0 0 0</pose>
+        <!-- <pose>-0.064 0 0.121 0 0 0</pose> -->
+        <pose>-0.064 0 0 0 0 0</pose>
         <update_rate>5</update_rate>
         <topic> ${prefix}_lidar </topic>

File: src/final_project/urdf/waffle.xacro (robot description, xacro)
@@ -167,6 +167,6 @@
         <parent link="base_link"/>
         <child link="base_scan"/>
-        <!-- <origin xyz="-0.064 0 0.122" rpy="0 0 0"/> -->
-        <origin xyz="-0.064 0 0" rpy="0 0 0"/>
+        <origin xyz="-0.064 0 0.122" rpy="0 0 0"/>
+        <!-- <origin xyz="-0.064 0 0" rpy="0 0 0"/> -->
     </joint>
     <link name="base_scan">
