Commit message: bot world and launch file added

File: final_project/urdf/burger.urdf (robot description, URDF)
Before this commit: robot waffle, 13 links, 12 joints
Links:
- removed link camera_depth_frame
- removed link camera_depth_optical_frame
- removed link camera_link
- removed link camera_rgb_frame
- removed link camera_rgb_optical_frame
- removed link caster_back_left_link
- removed link caster_back_right_link
- added link caster_back_link, mass 0.005; collision box size=0.030 0.009 0.020
- link base_link: mass 1.3729096e+00 -> 8.2573504e-01; geometry collision box size=0.140 0.140 0.143; visual mesh filename=file:///home/jimliu/Desktop/RSP_final_project/install/final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 scale=0.001 0.001 0.001
Joints:
- removed joint camera_depth_joint
- removed joint camera_depth_optical_joint
- removed joint camera_joint
- removed joint camera_rgb_joint
- removed joint camera_rgb_optical_joint
- removed joint caster_back_left_joint
- removed joint caster_back_right_joint
- added joint caster_back_joint: type fixed, parent base_link, child caster_back_link, origin xyz=-0.081 0 -0.004 rpy=-1.57 0 0
- joint base_joint: origin xyz=0 0 0.010 rpy=0 0 0 -> xyz=0.0 0.0 0.010 rpy=0 0 0
- joint imu_joint: origin xyz=0.0 0 0.068 rpy=0 0 0 -> xyz=-0.032 0 0.068 rpy=0 0 0
- joint scan_joint: origin xyz=-0.064 0 0.122 rpy=0 0 0 -> xyz=-0.032 0 0.172 rpy=0 0 0
- joint wheel_left_joint: origin xyz=0.0 0.144 0.023 rpy=-1.57 0 0 -> xyz=0.0 0.08 0.023 rpy=-1.57 0 0
- joint wheel_right_joint: origin xyz=0.0 -0.144 0.023 rpy=-1.57 0 0 -> xyz=0.0 -0.080 0.023 rpy=-1.57 0 0

File: final_project/urdf/burger.urdf.xacro (robot description, xacro)
@@ -1,13 +1,20 @@
 <robot xmlns:xacro="http://www.ros.org/wiki/xacro"  name="burger">
   <xacro:arg name="entity_name" default="burger"/>
-  <xacro:include filename="$(find final_project)/urdf/waffle.xacro" />
+  <xacro:include filename="$(find final_project)/urdf/burger.xacro" />
   <xacro:include filename="$(find final_project)/urdf/imu.xacro" />
   <xacro:include filename="$(find final_project)/urdf/lidar.xacro" />
-  <xacro:include filename="$(find final_project)/urdf/camera.xacro" />
+  <!-- <xacro:include filename="$(find final_project)/urdf/camera.xacro" /> -->
   <xacro:include filename="$(find final_project)/urdf/turtlebot3_plugin.xacro" />
-  <xacro:waffle prefix="$(arg entity_name)"/>
+  <!-- uncomment the next two lines if only spawn burger! -->
+  <!-- <xacro:include filename="$(find final_project)/urdf/ignition_system_plugin.xacro" />-->
+  <!-- <xacro:ignition_system_plugin/>-->
+  <xacro:burger prefix="$(arg entity_name)"/>
   <xacro:waffle_imu prefix="$(arg entity_name)"/>
-  <xacro:waffle_lidar prefix="$(arg entity_name)"/>
-  <xacro:waffle_camera prefix="$(arg entity_name)"/>
-  <xacro:turtlebot3_plugin entity_name="$(arg entity_name)"/>
+  <xacro:waffle_lidar prefix="$(arg entity_name)">
+    <pose>-0.032 0 0 0 0 0</pose>
+  </xacro:waffle_lidar>
+  <!-- <xacro:waffle_camera prefix="$(arg entity_name)"/> -->
+  <xacro:turtlebot3_plugin entity_name="$(arg entity_name)">
+    <wheel_separation>0.160</wheel_separation>
+  </xacro:turtlebot3_plugin>
 </robot>

Commit message: Adding world to launch files

File: final_project/urdf/burger.urdf (robot description, URDF)
Before this commit: robot burger, 7 links, 6 joints
Links:
- link base_link: geometry collision box size=0.140 0.140 0.143; visual mesh filename=file:///home/nivya/Desktop/RSP_final_project/install/final_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 scale=0.001 0.001 0.001
- link base_scan: geometry collision cylinder length=0.0315 radius=0.055; visual mesh filename=file:///home/nivya/Desktop/RSP_final_project/install/final_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 scale=0.001 0.001 0.001
- link wheel_left_link: geometry collision cylinder length=0.018 radius=0.033; visual mesh filename=file:///home/nivya/Desktop/RSP_final_project/install/final_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 scale=0.001 0.001 0.001
- link wheel_right_link: geometry collision cylinder length=0.018 radius=0.033; visual mesh filename=file:///home/nivya/Desktop/RSP_final_project/install/final_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 scale=0.001 0.001 0.001
