Commit message: joint state publishers modified

File: final_project/urdf/waffle.xacro (robot description, xacro)
@@ -61,10 +61,4 @@
         </inertial>
     </link>
-    <joint name="wheel_left_joint" type="continuous">
-        <parent link="base_link"/>
-        <child link="wheel_left_link"/>
-        <origin xyz="0.0 0.144 0.023" rpy="-1.57 0 0"/>
-        <axis xyz="0 0 1"/>
-    </joint>
     <link name="wheel_left_link">
         <visual>
@@ -89,4 +83,10 @@
         </inertial>
     </link>
+    <joint name="wheel_left_joint" type="continuous">
+        <parent link="base_link"/>
+        <child link="wheel_left_link"/>
+        <origin xyz="0.0 0.144 0.023" rpy="-1.57 0 0"/>
+        <axis xyz="0 0 1"/>
+    </joint>
     <joint name="wheel_right_joint" type="continuous">
         <parent link="base_link"/>
