Commit message: Navigation sort of work. Cannot get rid of odom warning

File: final_project/urdf/burger.urdf.xacro (robot description, xacro)
@@ -1,13 +1,17 @@
 <robot xmlns:xacro="http://www.ros.org/wiki/xacro"  name="burger">
   <xacro:arg name="entity_name" default="burger"/>
-  <xacro:include filename="$(find final_project)/urdf/waffle.xacro" />
+  <xacro:include filename="$(find final_project)/urdf/burger.xacro" />
   <xacro:include filename="$(find final_project)/urdf/imu.xacro" />
   <xacro:include filename="$(find final_project)/urdf/lidar.xacro" />
-  <xacro:include filename="$(find final_project)/urdf/camera.xacro" />
+  <!-- <xacro:include filename="$(find final_project)/urdf/camera.xacro" /> -->
   <xacro:include filename="$(find final_project)/urdf/turtlebot3_plugin.xacro" />
-  <xacro:waffle prefix="$(arg entity_name)"/>
+  <xacro:burger prefix="$(arg entity_name)"/>
   <xacro:waffle_imu prefix="$(arg entity_name)"/>
-  <xacro:waffle_lidar prefix="$(arg entity_name)"/>
-  <xacro:waffle_camera prefix="$(arg entity_name)"/>
-  <xacro:turtlebot3_plugin entity_name="$(arg entity_name)"/>
+  <xacro:waffle_lidar prefix="$(arg entity_name)">
+    <pose>-0.032 0 0.171 0 0 0</pose>
+  </xacro:waffle_lidar>
+  <!-- <xacro:waffle_camera prefix="$(arg entity_name)"/> -->
+  <xacro:turtlebot3_plugin entity_name="$(arg entity_name)">
+    <wheel_separation>0.160</wheel_separation>
+  </xacro:turtlebot3_plugin>
 </robot>

File: final_project/urdf/lidar.xacro (robot description, xacro)
@@ -1,4 +1,4 @@
 <robot xmlns:xacro="http://www.ros.org/wiki/xacro">
-  <xacro:macro name="waffle_lidar" params="prefix">
+  <xacro:macro name="waffle_lidar" params="prefix *pose">
     <gazebo reference="base_scan">
       <sensor type="gpu_lidar" name="${prefix}_lidar">
@@ -6,5 +6,6 @@
         <visualize>true</visualize>
         <!-- <pose>-0.064 0 0.121 0 0 0</pose> -->
-        <pose>-0.064 0 0 0 0 0</pose>
+        <!-- <pose>-0.064 0 0 0 0 0</pose> -->
+        <xacro:insert_block name="pose"/>
         <update_rate>5</update_rate>
         <topic> ${prefix}_lidar </topic>

File: final_project/urdf/turtlebot3_plugin.xacro (robot description, xacro)
@@ -1,4 +1,4 @@
 <robot xmlns:xacro="http://www.ros.org/wiki/xacro">
-  <xacro:macro name="turtlebot3_plugin" params="entity_name">
+  <xacro:macro name="turtlebot3_plugin" params="entity_name *wheel_separation">
     <gazebo>
       <plugin name="ignition::gazebo::systems::DiffDrive" filename="ignition-gazebo-diff-drive-system">
@@ -11,5 +11,6 @@
         <right_joint>wheel_right_joint</right_joint>
         <!-- kinematics -->
-        <wheel_separation>0.287</wheel_separation>
+        <!-- <wheel_separation>0.287</wheel_separation> -->
+        <xacro:insert_block name="wheel_separation"/>
         <!-- <wheel_diameter>0.066</wheel_diameter> -->
         <wheel_radius>0.033</wheel_radius>

File: final_project/urdf/waffle.urdf.xacro (robot description, xacro)
@@ -9,7 +9,11 @@
   <xacro:waffle prefix="$(arg entity_name)"/>
   <xacro:waffle_imu prefix="$(arg entity_name)"/>
-  <xacro:waffle_lidar prefix="$(arg entity_name)"/>
+  <xacro:waffle_lidar prefix="$(arg entity_name)">
+    <pose>-0.064 0 0 0 0 0</pose>
+  </xacro:waffle_lidar>
   <xacro:waffle_camera prefix="$(arg entity_name)"/>
-  <xacro:turtlebot3_plugin entity_name="$(arg entity_name)"/>
   <xacro:ignition_system_plugin/>
+  <xacro:turtlebot3_plugin entity_name="$(arg entity_name)">
+    <wheel_separation>0.287</wheel_separation>
+  </xacro:turtlebot3_plugin>
 </robot>

Commit message: burger xacro files are ready to use. missing camera

File: final_project/urdf/burger.urdf.xacro (robot description, xacro)
@@ -6,4 +6,7 @@
   <!-- <xacro:include filename="$(find final_project)/urdf/camera.xacro" /> -->
   <xacro:include filename="$(find final_project)/urdf/turtlebot3_plugin.xacro" />
+  <!-- uncomment the next two lines if only spawn burger! -->
+  <!-- <xacro:include filename="$(find final_project)/urdf/ignition_system_plugin.xacro" /> -->
+  <!-- <xacro:ignition_system_plugin/> -->
   <xacro:burger prefix="$(arg entity_name)"/>
   <xacro:waffle_imu prefix="$(arg entity_name)"/>

File: final_project/urdf/burger.xacro (robot description, xacro)
@@ -1,241 +1,162 @@
 <robot xmlns:xacro="http://www.ros.org/wiki/xacro">
   <xacro:macro name="burger" params="prefix">
-    <pose>0.0 0.0 0.0 0.0 0.0 0.0</pose>
+    <!-- Init colour -->
+    <material name="black">
+        <color rgba="0.0 0.0 0.0 1.0"/>
+    </material>
+    <material name="dark">
+        <color rgba="0.3 0.3 0.3 1.0"/>
+    </material>
+    <material name="light_black">
+        <color rgba="0.4 0.4 0.4 1.0"/>
+    </material>
+    <material name="blue">
+        <color rgba="0.0 0.0 0.8 1.0"/>
+    </material>
+    <material name="green">
+        <color rgba="0.0 0.8 0.0 1.0"/>
+    </material>
+    <material name="grey">
+        <color rgba="0.5 0.5 0.5 1.0"/>
+    </material>
+    <material name="orange">
+        <color rgba="1.0 0.4235 0.0392 1.0"/>
+    </material>
+    <material name="brown">
+        <color rgba="0.8706 0.8118 0.7647 1.0"/>
+    </material>
+    <material name="red">
+        <color rgba="0.8 0.0 0.0 1.0"/>
+    </material>
+    <material name="white">
+        <color rgba="1.0 1.0 1.0 1.0"/>
+    </material>
     <link name="base_footprint"/>
+    <joint name="base_joint" type="fixed">
+      <parent link="base_footprint"/>
+      <child link="base_link"/>
+      <origin xyz="0.0 0.0 0.010" rpy="0 0 0"/>
+    </joint>
     <link name="base_link">
-      <inertial>
-        <pose>-0.032 0 0.070 0 0 0</pose>
-        <inertia>
-          <ixx>7.2397393e-01</ixx>
-          <ixy>4.686399e-10</ixy>
-          <ixz>-1.09525703e-08</ixz>
-          <iyy>7.2397393e-01</iyy>
-          <iyz>2.8582649e-09</iyz>
-          <izz>6.53050163e-01</izz>
-        </inertia>
-        <mass>8.2573504e-01</mass>
-      </inertial>
-      <collision name="base_collision">
-        <pose>-0.032 0 0.070 0 0 0</pose>
-        <geometry>
-          <box>
-            <size>0.140 0.140 0.140</size>
-          </box>
-        </geometry>
-      </collision>
-      <visual name="base_visual">
-        <pose>-0.032 0 0 0 0 0</pose>
+      <visual>
+        <origin xyz="-0.032 0 0.0" rpy="0 0 0"/>
         <geometry>
           <mesh filename="file://$(find final_project)/models/turtlebot3_common/meshes/burger_base.dae" scale="0.001 0.001 0.001"/>
         </geometry>
+        <material name="light_black"/>
       </visual>
-    </link>
-    <link name="imu_link">
-    </link>
-    <link name="base_scan">
-      <inertial>
-        <pose>-0.020 0 0.161 0 0 0</pose>
-        <inertia>
-          <ixx>0.001</ixx>
-          <ixy>0.000</ixy>
-          <ixz>0.000</ixz>
-          <iyy>0.001</iyy>
-          <iyz>0.000</iyz>
-          <izz>0.001</izz>
-        </inertia>
-        <mass>0.114</mass>
-      </inertial>
-      <collision name="lidar_sensor_collision">
-        <pose>-0.020 0 0.161 0 0 0</pose>
+      <collision>
+        <origin xyz="-0.032 0 0.070" rpy="0 0 0"/>
         <geometry>
-          <cylinder>
-            <radius>0.0508</radius>
-            <length>0.055</length>
-          </cylinder>
+          <box size="0.140 0.140 0.143"/>
         </geometry>
       </collision>
-      <visual name="lidar_sensor_visual">
-        <pose>-0.032 0 0.171 0 0 0</pose>
+      <inertial>
+        <origin xyz="0 0 0" rpy="0 0 0"/>
+        <mass value="8.2573504e-01"/>
+        <inertia ixx="2.2124416e-03" ixy="-1.2294101e-05" ixz="3.4938785e-05" iyy="2.1193702e-03" iyz="-5.0120904e-06" izz="2.0064271e-03" />
+      </inertial>
+    </link>
+    <joint name="wheel_left_joint" type="continuous">
+      <parent link="base_link"/>
+      <child link="wheel_left_link"/>
+      <origin xyz="0.0 0.08 0.023" rpy="-1.57 0 0"/>
+      <axis xyz="0 0 1"/>
+    </joint>
+    <link name="wheel_left_link">
+      <visual>
+        <origin xyz="0 0 0" rpy="1.57 0 0"/>
+        <geometry>
+          <mesh filename="file://$(find final_project)/models/turtlebot3_common/meshes/tire.dae" scale="0.001 0.001 0.001"/>
+        </geometry>
+        <material name="dark"/>
+      </visual>
+      <collision>
+        <origin xyz="0 0 0" rpy="0 0 0"/>
+        <geometry>
+          <cylinder length="0.018" radius="0.033"/>
+        </geometry>
+      </collision>
+      <inertial>
+        <origin xyz="0 0 0" />
+        <mass value="2.8498940e-02" />
+        <inertia ixx="1.1175580e-05" ixy="-4.2369783e-11" ixz="-5.9381719e-09" iyy="1.1192413e-05" iyz="-1.4400107e-11" izz="2.0712558e-05" />
+      </inertial>
+    </link>
+    <joint name="wheel_right_joint" type="continuous">
+      <parent link="base_link"/>
+      <child link="wheel_right_link"/>
+      <origin xyz="0.0 -0.080 0.023" rpy="-1.57 0 0"/>
+      <axis xyz="0 0 1"/>
+    </joint>
+    <link name="wheel_right_link">
+      <visual>
+        <origin xyz="0 0 0" rpy="1.57 0 0"/>
+        <geometry>
+          <mesh filename="file://$(find final_project)/models/turtlebot3_common/meshes/tire.dae" scale="0.001 0.001 0.001"/>
+        </geometry>
+        <material name="dark"/>
+      </visual>
+      <collision>
+        <origin xyz="0 0 0" rpy="0 0 0"/>
+        <geometry>
+          <cylinder length="0.018" radius="0.033"/>
+        </geometry>
+      </collision>
+      <inertial>
+        <origin xyz="0 0 0" />
+        <mass value="2.8498940e-02" />
+        <inertia ixx="1.1175580e-05" ixy="-4.2369783e-11" ixz="-5.9381719e-09" iyy="1.1192413e-05" iyz="-1.4400107e-11" izz="2.0712558e-05" />
+      </inertial>
+    </link>
+    <joint name="caster_back_joint" type="fixed">
+      <parent link="base_link"/>
+      <child link="caster_back_link"/>
+      <origin xyz="-0.081 0 -0.004" rpy="-1.57 0 0"/>
+    </joint>
+    <link name="caster_back_link">
+      <collision>
+        <origin xyz="0 0.001 0" rpy="0 0 0"/>
+        <geometry>
+          <box size="0.030 0.009 0.020"/>
+        </geometry>
+      </collision>
+      <inertial>
+        <origin xyz="0 0 0" />
+        <mass value="0.005" />
+        <inertia ixx="0.001" ixy="0.0" ixz="0.0" iyy="0.001" iyz="0.0" izz="0.001" />
+      </inertial>
+    </link>
+    <joint name="imu_joint" type="fixed">
+      <parent link="base_link"/>
+      <child link="imu_link"/>
+      <origin xyz="-0.032 0 0.068" rpy="0 0 0"/>
+    </joint>
+    <link name="imu_link"/>
+    <joint name="scan_joint" type="fixed">
+      <parent link="base_link"/>
+      <child link="base_scan"/>
+      <origin xyz="-0.032 0 0.172" rpy="0 0 0"/>
+    </joint>
+    <link name="base_scan">
+      <visual>
+        <origin xyz="0 0 0.0" rpy="0 0 0"/>
         <geometry>
           <mesh filename="file://$(find final_project)/models/turtlebot3_common/meshes/lds.dae" scale="0.001 0.001 0.001"/>
         </geometry>
+        <material name="dark"/>
       </visual>
+      <collision>
+        <origin xyz="0.015 0 -0.0065" rpy="0 0 0"/>
+        <geometry>
+          <cylinder length="0.0315" radius="0.055"/>
+        </geometry>
+      </collision>
+      <inertial>
+        <mass value="0.114" />
+        <origin xyz="0 0 0" />
+        <inertia ixx="0.001" ixy="0.0" ixz="0.0" iyy="0.001" iyz="0.0" izz="0.001" />
+      </inertial>
     </link>
-    <link name="wheel_left_link">
-      <inertial>
-        <pose>0 0.08 0.023 -1.57 0 0</pose>
-        <inertia>
-          <ixx>1.8158194e-03</ixx>
-          <ixy>-9.3392e-12</ixy>
-          <ixz>1.04909e-11</ixz>
-          <iyy>3.2922126e-03</iyy>
-          <iyz>5.75694e-11</iyz>
-          <izz>1.8158194e-03</izz>
-        </inertia>
-        <mass>2.8498940e-02</mass>
-      </inertial>
-      <collision name="wheel_left_collision">
-        <pose>0 0.08 0.023 -1.57 0 0</pose>
-        <geometry>
-          <cylinder>
-            <radius>0.033</radius>
-            <length>0.018</length>
-          </cylinder>
-        </geometry>
-        <surface>
-          <!-- This friction pamareter don't contain reliable data!! -->
-          <friction>
-            <ode>
-              <mu>100000.0</mu>
-              <mu2>100000.0</mu2>
-              <fdir1>0 0 0</fdir1>
-              <slip1>0.0</slip1>
-              <slip2>0.0</slip2>
-            </ode>
-          </friction>
-          <contact>
-            <ode>
-              <soft_cfm>0</soft_cfm>
-              <soft_erp>0.2</soft_erp>
-              <kp>1e+5</kp>
-              <kd>1</kd>
-              <max_vel>0.01</max_vel>
-              <min_depth>0.001</min_depth>
-            </ode>
-          </contact>
-        </surface>
-      </collision>
-      <visual name="wheel_left_visual">
-        <pose>0 0.08 0.023 0 0 0</pose>
-        <geometry>
-          <mesh filename="file://$(find final_project)/models/turtlebot3_common/meshes/tire.dae" scale="0.001 0.001 0.001"/>
-        </geometry>
-      </visual>
-    </link>
-    <link name="wheel_right_link">
-      <inertial>
-        <pose>0.0 -0.08 0.023 -1.57 0 0</pose>
-        <inertia>
-          <ixx>1.8158194e-03</ixx>
-          <ixy>-9.3392e-12</ixy>
-          <ixz>1.04909e-11</ixz>
-          <iyy>3.2922126e-03</iyy>
-          <iyz>5.75694e-11</iyz>
-          <izz>1.8158194e-03</izz>
-        </inertia>
-        <mass>2.8498940e-02</mass>
-      </inertial>
-      <collision name="wheel_right_collision">
-        <pose>0.0 -0.08 0.023 -1.57 0 0</pose>
-        <geometry>
-          <cylinder>
-            <radius>0.033</radius>
-            <length>0.018</length>
-          </cylinder>
-        </geometry>
-        <surface>
-          <!-- This friction pamareter don't contain reliable data!! -->
-          <friction>
-            <ode>
-              <mu>100000.0</mu>
-              <mu2>100000.0</mu2>
-              <fdir1>0 0 0</fdir1>
-              <slip1>0.0</slip1>
-              <slip2>0.0</slip2>
-            </ode>
-          </friction>
-          <contact>
-            <ode>
-              <soft_cfm>0</soft_cfm>
-              <soft_erp>0.2</soft_erp>
-              <kp>1e+5</kp>
-              <kd>1</kd>
-              <max_vel>0.01</max_vel>
-              <min_depth>0.001</min_depth>
-            </ode>
-          </contact>
-        </surface>
-      </collision>
-      <visual name="wheel_right_visual">
-        <pose>0.0 -0.08 0.023 0 0 0</pose>
-        <geometry>
-          <mesh filename="file://$(find final_project)/models/turtlebot3_common/meshes/tire.dae" scale="0.001 0.001 0.001"/>
-        </geometry>
-      </visual>
-    </link>
-    <link name='caster_back_link'>
-      <pose>-0.081 0 -0.004 -1.57 0 0</pose>
-      <inertial>
-        <mass>0.005</mass>
-        <inertia>
-          <ixx>0.001</ixx>
-          <ixy>0.000</ixy>
-          <ixz>0.000</ixz>
-          <iyy>0.001</iyy>
-          <iyz>0.000</iyz>
-          <izz>0.001</izz>
-        </inertia>
-      </inertial>
-      <collision name='collision'>
-        <geometry>
-          <sphere>
-            <radius>0.005000</radius>
-          </sphere>
-        </geometry>
-        <surface>
-          <contact>
-            <ode>
-              <soft_cfm>0</soft_cfm>
-              <soft_erp>0.2</soft_erp>
-              <kp>1e+5</kp>
-              <kd>1</kd>
-              <max_vel>0.01</max_vel>
-              <min_depth>0.001</min_depth>
-            </ode>
-          </contact>
-        </surface>
-      </collision>
-    </link>
-    <joint name="base_joint" type="fixed">
-      <parent>base_footprint</parent>
-      <child>base_link</child>
-      <pose>0.0 0.0 0.010 0 0 0</pose>
-    </joint>
-    <joint name="wheel_left_joint" type="revolute">
-      <parent>base_link</parent>
-      <child>wheel_left_link</child>
-      <pose>0.0 0.08 0.023 -1.57 0 0</pose>
-      <axis>
-        <xyz>0 0 1</xyz>
-      </axis>
-    </joint>
-    <joint name="wheel_right_joint" type="revolute">
-      <parent>base_link</parent>
-      <child>wheel_right_link</child>
-      <pose>0.0 -0.08 0.023 -1.57 0 0</pose>
-      <axis>
-        <xyz>0 0 1</xyz>
-      </axis>
-    </joint>
-    <joint name='caster_back_joint' type='ball'>
-      <parent>base_link</parent>
-      <child>caster_back_link</child>
-    </joint>
-    <joint name="imu_joint" type="fixed">
-      <parent>base_link</parent>
-      <child>imu_link</child>
-      <pose>-0.032 0 0.068 0 0 0</pose>
-      <axis>
-        <xyz>0 0 1</xyz>
-      </axis>
-    </joint>
-    <joint name="lidar_joint" type="fixed">
-      <parent>base_link</parent>
-      <child>base_scan</child>
-      <pose>-0.032 0 0.171 0 0 0</pose>
-      <axis>
-        <xyz>0 0 1</xyz>
-      </axis>
-    </joint>
   </xacro:macro>
 </robot>

Commit message: add camera to burger and bridge image topic

File: final_project/urdf/burger.urdf.xacro (robot description, xacro)
@@ -3,5 +3,5 @@
   <xacro:include filename="$(find final_project)/urdf/burger.xacro" />
   <xacro:include filename="$(find final_project)/urdf/imu.xacro" />
-  <!-- <xacro:include filename="$(find final_project)/urdf/camera.xacro" /> -->
+  <xacro:include filename="$(find final_project)/urdf/camera.xacro" />
   <xacro:include filename="$(find final_project)/urdf/turtlebot3_plugin_burger.xacro" />
   <!-- uncomment the next two lines if only spawn burger! -->
@@ -10,5 +10,5 @@
   <xacro:burger prefix="$(arg entity_name)"/>
   <xacro:waffle_imu prefix="$(arg entity_name)"/>
-  <!-- <xacro:waffle_camera prefix="$(arg entity_name)"/> -->
+  <xacro:waffle_camera prefix="$(arg entity_name)"/>
   <xacro:turtlebot3_plugin entity_name="$(arg entity_name)">
     <wheel_separation>0.160</wheel_separation>

File: final_project/urdf/burger.xacro (robot description, xacro)
@@ -159,4 +159,59 @@
       </inertial>
     </link>
+    <joint name="camera_joint" type="fixed">
+        <origin xyz="0.036 -0.035 0.094" rpy="0 0 0"/>
+        <parent link="base_link"/>
+        <child link="camera_link"/>
+    </joint>
+    <!-- burger camera customization -->
+    <link name="camera_link">
+        <visual>
+        <origin xyz="0 0 0" rpy="1.57 0 1.57"/>
+        <geometry>
+        <mesh filename="file://$(find final_project)/models/turtlebot3_common/meshes/r200.dae" scale="0.5 0.5 0.5"/>
+        </geometry>
+        </visual>
+        <collision>
+        <origin xyz="0.003 0.065 0.007" rpy="0 0 0"/>
+        <geometry>
+            <box size="0.008 0.132 0.020"/>
+        </geometry>
+        </collision>
+        <!-- This inertial field needs doesn't contain reliable data!! -->
+    <!--   <inertial>
+        <mass value="0.564" />
+        <origin xyz="0 0 0" />
+        <inertia ixx="0.003881243" ixy="0.0" ixz="0.0"
+                iyy="0.000498940" iyz="0.0"
+                izz="0.003879257" />
+        </inertial>-->
+    </link>
+    <joint name="camera_rgb_joint" type="fixed">
+        <origin xyz="0.005 0.018 0.013" rpy="0 0 0"/>
+        <!-- <origin xyz="${r200_cam_rgb_px} ${r200_cam_rgb_py} ${r200_cam_rgb_pz}" rpy="0 0 0"/> -->
+        <parent link="camera_link"/>
+        <child link="camera_rgb_frame"/>
+    </joint>
+    <link name="camera_rgb_frame">
+    </link>
+    <joint name="camera_rgb_optical_joint" type="fixed">
+        <origin xyz="0 0 0" rpy="-1.57 0 -1.57"/>
+        <parent link="camera_rgb_frame"/>
+        <child link="camera_rgb_optical_frame"/>
+    </joint>
+    <link name="camera_rgb_optical_frame"/>
+    <joint name="camera_depth_joint" type="fixed">
+        <origin xyz="0.005 0.028 0.013" rpy="0 0 0"/>
+        <!-- <origin xyz="${r200_cam_rgb_px} ${r200_cam_rgb_py + r200_cam_depth_offset} ${r200_cam_rgb_pz}" rpy="0 0 0"/> -->
+        <parent link="camera_link"/>
+        <child link="camera_depth_frame"/>
+    </joint>
+    <link name="camera_depth_frame"/>
+    <joint name="camera_depth_optical_joint" type="fixed">
+        <origin xyz="0 0 0" rpy="-1.57 0 -1.57"/>
+        <parent link="camera_depth_frame"/>
+        <child link="camera_depth_optical_frame"/>
+    </joint>
+    <link name="camera_depth_optical_frame"/>
   </xacro:macro>
 </robot>
