Commit message: multibots

File: final_project/urdf/waffle.urdf.xacro (robot description, xacro)
@@ -4,5 +4,5 @@
   <xacro:include filename="$(find final_project)/urdf/imu.xacro" />
   <xacro:include filename="$(find final_project)/urdf/lidar.xacro" />
-  <xacro:include filename="$(find final_project)/urdf/camera.xacro" />
+  <!-- <xacro:include filename="$(find final_project)/urdf/camera.xacro" /> -->
   <xacro:include filename="$(find final_project)/urdf/turtlebot3_plugin.xacro" />
   <xacro:include filename="$(find final_project)/urdf/ignition_system_plugin.xacro" />
@@ -12,5 +12,5 @@
     <pose>-0.064 0 0 0 0 0</pose>
   </xacro:waffle_lidar>
-  <xacro:waffle_camera prefix="$(arg entity_name)"/>
+  <!-- <xacro:waffle_camera prefix="$(arg entity_name)"/> -->
   <xacro:ignition_system_plugin/>
   <xacro:turtlebot3_plugin entity_name="$(arg entity_name)">

File: ign_gazebo/urdf/bot_world.xacro (robot description, xacro)
@@ -152,4 +152,5 @@
 		</link>
     <xacro:box_world name="box_2" parent="base_box">
+    	<!-- <origin xyz="-0.431 0 0" rpy="0 0 1.57"/> -->
     	<origin xyz="-0.431 0 0" rpy="0 0 1.57"/>
     </xacro:box_world>
