Commit message: merge all branchs

File: ign_gazebo/urdf/bot_world.urdf (robot description, URDF)
Before this commit: robot aruco_markers, 12 links, 11 joints
Links:
- removed link box_1
- removed link box_3
- link marker01_link: geometry collision box size=0.1 0.1 0.1; visual mesh filename=file:///home/huan/RSP_final_project/install/ign_gazebo/shar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 scale=0.25 0.25 0.25
- link marker03_link: geometry collision box size=0.1 0.1 0.1; visual mesh filename=file:///home/huan/RSP_final_project/install/ign_gazebo/shar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 scale=0.25 0.25 0.25
- link shelf_link: geometry collision box size=4.5 0.6 1.8; visual mesh filename=file:///home/huan/RSP_final_project/install/ign_gazebo/shar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 scale=0.2 0.3 0.3
Joints:
- removed joint box_1_joint
- removed joint box_3_joint

File: ign_gazebo/urdf/bot_world.xacro (robot description, xacro)
@@ -81,5 +81,5 @@
 			</inertial>
 		</link>
-		<joint name="${name}_joint" type="continuous">
+		<joint name="${name}_joint" type="fixed">
 			<xacro:insert_block name="origin" />
 			<parent link="${parent}"/>
@@ -151,15 +151,9 @@
 			</inertial>
 		</link>
-    <xacro:box_world name="box_1" parent="base_box">
-    	<origin xyz="0.42 0 0" rpy="0 0 1.57"/>
-    </xacro:box_world>
     <xacro:box_world name="box_2" parent="base_box">
-    	<origin xyz="-0.42 0 0" rpy="0 0 1.57"/>
-    </xacro:box_world>
-    <xacro:box_world name="box_3" parent="base_box">
-    	<origin xyz="-0.21 -0.1275 0" rpy="0 0 1.57"/>
+    	<origin xyz="-0.431 0 0" rpy="0 0 1.57"/>
     </xacro:box_world>
     <xacro:box_world name="box_4" parent="base_box">
-    	<origin xyz="-0.63 0 0" rpy="0 0 1.57"/>
+    	<origin xyz="-0.65 0 0" rpy="0 0 1.57"/>
     </xacro:box_world>
     <xacro:wall_world name="wall_1" parent="base_box">
