Commit message: draw maps

File: ign_gazebo/urdf/bot_world.xacro (robot description, xacro)
@@ -23,5 +23,5 @@
 			</collision>
 		</link>
-		<joint name="${name}_joint" type="continuous">
+		<joint name="${name}_joint" type="fixed">
 			<xacro:insert_block name="origin" />
 			<parent link="${parent}"/>
@@ -191,5 +191,5 @@
 			</inertial>
 		</link>
-		<joint name="wb1_w1_joint" type="continuous">
+		<joint name="wb1_w1_joint" type="fixed">
 			<origin xyz="3.2 0.0 1.0" rpy="0 0 0"/>
 			<parent link="base_box"/>
@@ -218,5 +218,5 @@
 			</inertial>
 		</link>
-		<joint name="wb1_w2_joint" type="continuous">
+		<joint name="wb1_w2_joint" type="fixed">
 			<origin xyz="1.4 2.7 1.0" rpy="0 0 1.57"/>
 			<parent link="base_box"/>

Commit message: update xacro

File: ign_gazebo/urdf/bot_world.xacro (robot description, xacro)
@@ -23,5 +23,5 @@
 			</collision>
 		</link>
-		<joint name="${name}_joint" type="continuous">
+		<joint name="${name}_joint" type="fixed">
 			<xacro:insert_block name="origin" />
 			<parent link="${parent}"/>
@@ -151,13 +151,13 @@
 			</inertial>
 		</link>
-    <xacro:box_world name="box_1" parent="base_box">
-    	<origin xyz="0.42 0 0" rpy="0 0 1.57"/>
-    </xacro:box_world>
+    <!-- <xacro:box_world name="box_1" parent="base_box"> -->
+    <!-- 	<origin xyz="0.42 0 0" rpy="0 0 1.57"/> -->
+    <!-- </xacro:box_world> -->
     <xacro:box_world name="box_2" parent="base_box">
     	<origin xyz="-0.42 0 0" rpy="0 0 1.57"/>
     </xacro:box_world>
-    <xacro:box_world name="box_3" parent="base_box">
-    	<origin xyz="-0.21 -0.1275 0" rpy="0 0 1.57"/>
-    </xacro:box_world>
+    <!-- <xacro:box_world name="box_3" parent="base_box"> -->
+    <!-- 	<origin xyz="-0.21 -0.1275 0" rpy="0 0 1.57"/> -->
+    <!-- </xacro:box_world> -->
     <xacro:box_world name="box_4" parent="base_box">
     	<origin xyz="-0.63 0 0" rpy="0 0 1.57"/>
@@ -191,5 +191,5 @@
 			</inertial>
 		</link>
-		<joint name="wb1_w1_joint" type="continuous">
+		<joint name="wb1_w1_joint" type="fixed">
 			<origin xyz="3.2 0.0 1.0" rpy="0 0 0"/>
 			<parent link="base_box"/>
@@ -218,5 +218,5 @@
 			</inertial>
 		</link>
-		<joint name="wb1_w2_joint" type="continuous">
+		<joint name="wb1_w2_joint" type="fixed">
 			<origin xyz="1.4 2.7 1.0" rpy="0 0 1.57"/>
 			<parent link="base_box"/>

Commit message: moving box fixed

File: ign_gazebo/urdf/bot_world.xacro (robot description, xacro)
@@ -81,5 +81,5 @@
 			</inertial>
 		</link>
-		<joint name="${name}_joint" type="continuous">
+		<joint name="${name}_joint" type="fixed">
 			<xacro:insert_block name="origin" />
 			<parent link="${parent}"/>
@@ -151,15 +151,9 @@
 			</inertial>
 		</link>
-    <!-- <xacro:box_world name="box_1" parent="base_box"> -->
-    <!-- 	<origin xyz="0.42 0 0" rpy="0 0 1.57"/> -->
-    <!-- </xacro:box_world> -->
     <xacro:box_world name="box_2" parent="base_box">
-    	<origin xyz="-0.42 0 0" rpy="0 0 1.57"/>
+    	<origin xyz="-0.431 0 0" rpy="0 0 1.57"/>
     </xacro:box_world>
-    <!-- <xacro:box_world name="box_3" parent="base_box"> -->
-    <!-- 	<origin xyz="-0.21 -0.1275 0" rpy="0 0 1.57"/> -->
-    <!-- </xacro:box_world> -->
     <xacro:box_world name="box_4" parent="base_box">
-    	<origin xyz="-0.63 0 0" rpy="0 0 1.57"/>
+    	<origin xyz="-0.65 0 0" rpy="0 0 1.57"/>
     </xacro:box_world>
     <xacro:wall_world name="wall_1" parent="base_box">

File: ign_gazebo/urdf/moving_box.urdf (robot description, URDF)
Before this commit: robot Moving_box, 2 links, 1 joints
Links:
- removed link world
- added link base_link
- link box_3: mass 0.01 -> 0.18
Joints:
- joint box_3_joint: axis 0 0 1 -> (none); origin xyz=-0.21 -0.1275 0 rpy=0 0 1.57 -> xyz=-0.215 -0.1275 0 rpy=0 0 1.57; parent world -> base_link; type planar -> fixed

File: ign_gazebo/urdf/moving_box.urdf.xacro (robot description, xacro)
@@ -1,9 +1,4 @@
 <robot xmlns:xacro="http://www.ros.org/wiki/xacro" name="Moving_box">
        <xacro:include filename="$(find ign_gazebo)/urdf/moving_box.xacro"/>
-       <link name = "world">
-           <origin xyz = "0 0 0" rpy = "0 0 0"/>
-       </link>
-    <xacro:box_world name="box_3" parent="world">
-    	<origin xyz="-0.21 -0.1275 0" rpy="0 0 1.57"/>
-    </xacro:box_world>
+       <xacro:box_world name="box_3"/>
 </robot>

File: ign_gazebo/urdf/moving_box.xacro (robot description, xacro)
@@ -1,10 +1,19 @@
 <robot xmlns:xacro="http://www.ros.org/wiki/xacro" name="Moving_box">
-	<xacro:macro name="box_world" params="name parent *origin">
+<xacro:macro name="box_world" params="name">
 		<xacro:property name="box_height" value="0.165"/>
 		<xacro:property name="box_width" value="0.21"/>
 		<xacro:property name="box_length" value="0.255"/>
+    <link name = "base_link">
+      <origin xyz="-0.215 -0.1275 0" rpy="0 0 1.57"/>
+    </link>
+		<joint name="${name}_joint" type="fixed">
+      <origin xyz="-0.215 -0.1275 0" rpy="0 0 1.57"/>
+			<parent link="base_link"/>
+			<child link="${name}"/>
+		</joint>
 		<link name="${name}">
 			<visual>
 				<origin xyz="0 0 ${0.5*box_height}" rpy="0 0 0"/>
+				<!-- <origin xyz="0 0 0" rpy="0 0 0"/> -->
 				<geometry>
 					<box size="${box_length} ${box_width} ${box_height}"/>
@@ -16,4 +25,5 @@
 			<collision>
 				<origin xyz="0 0 ${0.5*box_height}" rpy="0 0 0"/>
+				<!-- <origin xyz="0 0 0" rpy="0 0 0"/> -->
 				<geometry>
 					<box size="${box_length} ${box_width} ${box_height}"/>
@@ -22,14 +32,8 @@
 			<inertial>
 				<origin xyz="0 0 ${0.5*box_height}" rpy="0 0 0"/>
-				<mass value="0.01"/>
+				<mass value="0.18"/>
 				<inertia ixx="6.0e-4" ixy="0" ixz="0" iyy="6.0e-4" iyz="0" izz="6.0e-4"/>
 			</inertial>
 		</link>
-		<joint name="${name}_joint" type="planar">
-            <axis xyz= "0 0 1"/>
-			<xacro:insert_block name="origin" />
-			<parent link="${parent}"/>
-			<child link="${name}"/>
-		</joint>
 	</xacro:macro>
 </robot>

Commit message: moving box update

File: ign_gazebo/urdf/bot_world.xacro (robot description, xacro)
@@ -49,5 +49,5 @@
 			</collision>
 		</link>
-		<joint name="${name}_joint" type="continuous">
+		<joint name="${name}_joint" type="fixed">
 			<xacro:insert_block name="origin" />
 			<parent link="${parent}"/>
@@ -113,5 +113,5 @@
 			</inertial>
 		</link>
-		<joint name="${name}_joint" type="continuous">
+		<joint name="${name}_joint" type="fixed">
 		  <xacro:insert_block name="origin" />
 			<parent link="${parent}"/>
@@ -186,5 +186,5 @@
 		</link>
 		<joint name="wb1_w1_joint" type="fixed">
-			<origin xyz="3.2 0.0 1.0" rpy="0 0 0"/>
+			<origin xyz="3.2 0.0 0.5" rpy="0 0 0"/>
 			<parent link="base_box"/>
 			<child link="wb1_w1"/>
@@ -201,5 +201,6 @@
 			</visual>
 			<collision>
-				<origin xyz="0 0 0.1" rpy="0 0 0"/>
+				<!-- <origin xyz="0 0 0.1" rpy="0 0 0"/> -->
+                <origin xyz="3.2 0.0 0.5" rpy="0 0 0"/>
 				<geometry>
 					<box size="${wb_length} ${wb_width} ${wb_height}"/>

File: ign_gazebo/urdf/moving_box.urdf (robot description, URDF)
Before this commit: robot Moving_box, 2 links, 1 joints
Links:
- link box_3: mass 0.18 -> 1.3729096e+00

File: ign_gazebo/urdf/moving_box.urdf.xacro (robot description, xacro)
@@ -2,3 +2,11 @@
        <xacro:include filename="$(find ign_gazebo)/urdf/moving_box.xacro"/>
        <xacro:box_world name="box_3"/>
+      <link name = "base_link"/>
+      <joint name="box_3_joint" type="fixed">
+        <!-- <axis xyz = "1 0 0"/> -->
+        <origin xyz="-0.215 -0.1275 0" rpy="0 0 1.57"/>
+        <parent link="base_link"/>
+        <child link="box_3"/>
+        <!-- <limit lower= "-1" upper = "1" effort="100" velocity = ".2"/> -->
+      </joint>
 </robot>

File: ign_gazebo/urdf/moving_box.xacro (robot description, xacro)
@@ -4,12 +4,4 @@
 		<xacro:property name="box_width" value="0.21"/>
 		<xacro:property name="box_length" value="0.255"/>
-    <link name = "base_link">
-      <origin xyz="-0.215 -0.1275 0" rpy="0 0 1.57"/>
-    </link>
-		<joint name="${name}_joint" type="fixed">
-      <origin xyz="-0.215 -0.1275 0" rpy="0 0 1.57"/>
-			<parent link="base_link"/>
-			<child link="${name}"/>
-		</joint>
 		<link name="${name}">
 			<visual>
@@ -32,6 +24,8 @@
 			<inertial>
 				<origin xyz="0 0 ${0.5*box_height}" rpy="0 0 0"/>
-				<mass value="0.18"/>
-				<inertia ixx="6.0e-4" ixy="0" ixz="0" iyy="6.0e-4" iyz="0" izz="6.0e-4"/>
+        <mass value="1.3729096e+00"/>
+        <inertia ixx="8.7002718e-03" ixy="-4.7576583e-05" ixz="1.1160499e-04"
+                iyy="8.6195418e-03" iyz="-3.5422299e-06"
+                izz="1.4612727e-02" />
 			</inertial>
 		</link>

Commit message: moving box problem fixed

File: ign_gazebo/urdf/bot_world.xacro (robot description, xacro)
@@ -78,11 +78,35 @@
 				<origin xyz="0 0 ${0.5*box_height}" rpy="0 0 0"/>
 				<mass value="0.180"/>
-				<inertia ixx="6.0e-4" ixy="0" ixz="0" iyy="6.0e-4" iyz="0" izz="6.0e-4"/>
-			</inertial>
-		</link>
+				<inertia ixx="6.0e-3" ixy="0" ixz="0" iyy="6.0e-3" iyz="0" izz="6.0e-3"/>
+			</inertial>
+		</link>
+		<gazebo reference="${name}">
+    	   <surface>
+      		<friction>
+        		<ode>
+          			<mu>1</mu>
+          			<mu2>1</mu2>
+          			<slip1>0</slip1>
+          			<slip2>0</slip2>
+          			<fdir1>1 0 0 </fdir1>
+        		</ode>
+      		</friction>
+      		<contact>
+        		<ode>
+          			<soft_cfm>0</soft_cfm>
+          			<soft_erp>0.2</soft_erp>
+          			<kp>1e+13</kp>
+          			<kd>1</kd>
+          			<max_vel>0.01</max_vel>
+          			<min_depth>0</min_depth>
+        		</ode>
+      		</contact>
+    		</surface>
+    	</gazebo>
 		<joint name="${name}_joint" type="fixed">
 			<xacro:insert_block name="origin" />
 			<parent link="${parent}"/>
 			<child link="${name}"/>
+			<dynamics damping="0.1" friction="2" />
 		</joint>
 	</xacro:macro>
@@ -148,7 +172,30 @@
 				<origin xyz="0 0 ${0.5*box_height}" rpy="0 0 0"/>
 				<mass value="0.180"/>
-				<inertia ixx="6.0e-4" ixy="0" ixz="0" iyy="6.0e-4" iyz="0" izz="6.0e-4"/>
-			</inertial>
-		</link>
+				<inertia ixx="6.0e-3" ixy="0" ixz="0" iyy="6.0e-3" iyz="0" izz="6.0e-3"/>
+			</inertial>
+		</link>
+		<gazebo reference="base_box">
+    	   <surface>
+      		<friction>
+        		<ode>
+          			<mu>1</mu>
+          			<mu2>1</mu2>
+          			<slip1>0</slip1>
+          			<slip2>0</slip2>
+          			<fdir1>1 0 0 </fdir1>
+        		</ode>
+      		</friction>
+      		<contact>
+        		<ode>
+          			<soft_cfm>0</soft_cfm>
+          			<soft_erp>0.2</soft_erp>
+          			<kp>1e+13</kp>
+          			<kd>1</kd>
+          			<max_vel>0.01</max_vel>
+          			<min_depth>0</min_depth>
+        		</ode>
+      		</contact>
+    		</surface>
+    	</gazebo>
     <xacro:box_world name="box_2" parent="base_box">
     	<origin xyz="-0.431 0 0" rpy="0 0 1.57"/>
@@ -162,5 +209,5 @@
     <xacro:wall_world name="wall_2" parent="base_box">
     	<origin xyz="-0.1 2.8 0.0" rpy="0 0 1.57"/>
-		</xacro:wall_world>
+	</xacro:wall_world>
 		<link name="wb1_w1">
 			<visual>

File: ign_gazebo/urdf/moving_box.urdf.xacro (robot description, xacro)
@@ -2,11 +2,3 @@
        <xacro:include filename="$(find ign_gazebo)/urdf/moving_box.xacro"/>
        <xacro:box_world name="box_3"/>
-      <link name = "base_link"/>
-      <joint name="box_3_joint" type="fixed">
-        <!-- <axis xyz = "1 0 0"/> -->
-        <origin xyz="-0.215 -0.1275 0" rpy="0 0 1.57"/>
-        <parent link="base_link"/>
-        <child link="box_3"/>
-        <!-- <limit lower= "-1" upper = "1" effort="100" velocity = ".2"/> -->
-      </joint>
 </robot>

File: ign_gazebo/urdf/moving_box.xacro (robot description, xacro)
@@ -24,8 +24,6 @@
 			<inertial>
 				<origin xyz="0 0 ${0.5*box_height}" rpy="0 0 0"/>
-        <mass value="1.3729096e+00"/>
-        <inertia ixx="8.7002718e-03" ixy="-4.7576583e-05" ixz="1.1160499e-04"
-                iyy="8.6195418e-03" iyz="-3.5422299e-06"
-                izz="1.4612727e-02" />
+				<mass value="0.180"/>
+				<inertia ixx="2.0" ixy="0" ixz="0" iyy="2.0" iyz="0" izz="2.0"/>
 			</inertial>
 		</link>

Commit message: updated simulation

File: ign_gazebo/urdf/bot_world.xacro (robot description, xacro)
@@ -10,5 +10,5 @@
 				<origin xyz="0 0 0.0" rpy="0 1.57 0"/>
 				<geometry>
-					<mesh filename="file://$(find ign_gazebo)/meshes/${name}.stl" scale="0.25 0.25 0.25"/>
+					<mesh filename="file://$(find ign_gazebo)/meshes/${name}.stl" scale="0.6 0.6 0.6"/>
 				</geometry>
 				<material name="Gray">
@@ -122,5 +122,5 @@
 				</geometry>
 				<material name="Maroon">
-					<color rgba="0.5 0.0 0.0 1.0"/>
+					<color rgba="1 1 1 1"/>
 				</material>
 			</visual>
@@ -151,6 +151,6 @@
 		<xacro:property name="wall_length" value="0.2"/>
 		<xacro:property name="wb_length" value="0.1"/>
-		<xacro:property name="wb_width" value="0.2"/>
-		<xacro:property name="wb_height" value="0.2"/>
+		<xacro:property name="wb_width" value="0.6"/>
+		<xacro:property name="wb_height" value="0.6"/>
 		<link name="base_box">
 			<visual>
@@ -200,8 +200,8 @@
     <xacro:box_world name="box_2" parent="base_box">
     	<!-- <origin xyz="-0.431 0 0" rpy="0 0 1.57"/> -->
-    	<origin xyz="-0.431 0 0" rpy="0 0 1.57"/>
+    	<origin xyz="-0.48 0 0" rpy="0 0 1.57"/>
     </xacro:box_world>
     <xacro:box_world name="box_4" parent="base_box">
-    	<origin xyz="-0.65 0 0" rpy="0 0 1.57"/>
+    	<origin xyz="-0.71 0 0" rpy="0 0 1.57"/>
     </xacro:box_world>
     <xacro:wall_world name="wall_1" parent="base_box">

File: ign_gazebo/urdf/sample_moving_box.xacro (robot description, xacro)
@@ -28,5 +28,5 @@
 		</link>
 		<joint name="${name}_joint" type="fixed">
-			<origin xyz="-0.215 -0.265 0" rpy="0 0 1.57"/>
+			<origin xyz="-0.25 -0.265 0" rpy="0 0 1.57"/>
 			<parent link="moving_box_base"/>
 			<child link="${name}"/>

Commit message: still need to run client and server nodes

File: ign_gazebo/urdf/bot_world.xacro (robot description, xacro)
@@ -164,5 +164,5 @@
 			</visual>
 			<collision>
-				<origin xyz="0 0 ${0.5*box_height}" rpy="0 0 0"/>
+				<origin xyz="0 0 ${0.5*box_height}" rpy="0 0 1.57"/>
 				<geometry>
 					<box size="${box_length} ${box_width} ${box_height}"/>
@@ -200,8 +200,8 @@
     <xacro:box_world name="box_2" parent="base_box">
     	<!-- <origin xyz="-0.431 0 0" rpy="0 0 1.57"/> -->
-    	<origin xyz="-0.48 0 0" rpy="0 0 1.57"/>
+    	<origin xyz="-0.47 0 0" rpy="0 0 1.57"/>
     </xacro:box_world>
     <xacro:box_world name="box_4" parent="base_box">
-    	<origin xyz="-0.71 0 0" rpy="0 0 1.57"/>
+    	<origin xyz="-0.69 0 0" rpy="0 0 1.57"/>
     </xacro:box_world>
     <xacro:wall_world name="wall_1" parent="base_box">

File: ign_gazebo/urdf/sample_moving_box.xacro (robot description, xacro)
@@ -28,5 +28,5 @@
 		</link>
 		<joint name="${name}_joint" type="fixed">
-			<origin xyz="-0.25 -0.265 0" rpy="0 0 1.57"/>
+			<origin xyz="-0.24 -0.265 0" rpy="0 0 1.57"/>
 			<parent link="moving_box_base"/>
 			<child link="${name}"/>
