Commit message: split client

File: ign_gazebo/urdf/sample_moving_box.xacro (robot description, xacro)
@@ -28,5 +28,5 @@
 		</link>
 		<joint name="${name}_joint" type="fixed">
-			<origin xyz="-0.24 -0.265 0" rpy="0 0 1.57"/>
+			<origin xyz="-0.24 -0.2 0" rpy="0 0 1.57"/>
 			<parent link="moving_box_base"/>
 			<child link="${name}"/>
